Commit message: Bug fix for can_velocity_converter and tf

File: eagleye_util/tf/urdf/sensors.xacro (robot description, xacro)
@@ -3,5 +3,5 @@
   xmlns:xacro="http://ros.org/wiki/xacro">
   <xacro:arg name="config_dir" default="$(find eagleye_tf)"/>
-  <xacro:property name="calibration" value="${load_yaml('$(arg config_dir)/sensors_tf.yaml')}"/>
+  <xacro:property name="calibration" value="${load_yaml('$(arg config_dir)/config/sensors_tf.yaml')}"/>
   <xacro:property name="size" value="1" />
   <!-- base_link -->

Commit message: Fix incorrect names

File: eagleye_util/tf/urdf/sensors.xacro (robot description, xacro)
@@ -6,5 +6,5 @@
   <xacro:property name="size" value="1" />
   <!-- base_link -->
-  <link name="${calibration['basic_parent_flame']}">
+  <link name="${calibration['basic_parent_frame']}">
     <visual>
       <origin xyz="0 0 0" rpy="0 0 0"/>
@@ -26,5 +26,5 @@
     </link>
   </xacro:macro>
-  <xacro:imu parent="${calibration['basic_parent_flame']}" x="${calibration['base_link2imu']['x']}" y="${calibration['base_link2imu']['y']}" z="${calibration['base_link2imu']['z']}" roll="${calibration['base_link2imu']['roll']}" pitch="${calibration['base_link2imu']['pitch']}" yaw="${calibration['base_link2imu']['yaw']}" />
+  <xacro:imu parent="${calibration['basic_parent_frame']}" x="${calibration['base_link2imu']['x']}" y="${calibration['base_link2imu']['y']}" z="${calibration['base_link2imu']['z']}" roll="${calibration['base_link2imu']['roll']}" pitch="${calibration['base_link2imu']['pitch']}" yaw="${calibration['base_link2imu']['yaw']}" />
   <!-- gnss -->
   <xacro:macro name="gnss" params="parent x y z roll pitch yaw">
@@ -39,4 +39,4 @@
     </link>
   </xacro:macro>
-  <xacro:gnss parent="${calibration['basic_parent_flame']}" x="${calibration['base_link2gnss']['x']}" y="${calibration['base_link2gnss']['y']}" z="${calibration['base_link2gnss']['z']}" roll="${calibration['base_link2gnss']['roll']}" pitch="${calibration['base_link2gnss']['pitch']}" yaw="${calibration['base_link2gnss']['yaw']}" />
+  <xacro:gnss parent="${calibration['basic_parent_frame']}" x="${calibration['base_link2gnss']['x']}" y="${calibration['base_link2gnss']['y']}" z="${calibration['base_link2gnss']['z']}" roll="${calibration['base_link2gnss']['roll']}" pitch="${calibration['base_link2gnss']['pitch']}" yaw="${calibration['base_link2gnss']['yaw']}" />
 </robot>

Commit message: Param rename

File: eagleye_util/tf/urdf/sensors.xacro (robot description, xacro)
@@ -3,5 +3,5 @@
   xmlns:xacro="http://ros.org/wiki/xacro">
   <xacro:arg name="config_dir" default="$(find eagleye_tf)"/>
-  <xacro:property name="calibration" value="${load_yaml('$(arg config_dir)/config/sensors_tf.yaml')}"/>
+  <xacro:property name="calibration" value="${xacro.load_yaml,('$(arg config_dir)/config/sensors_tf.yaml')}"/>
   <xacro:property name="size" value="1" />
   <!-- base_link -->
